Commit message: Fix duplicate 'abb_orange' material definition in URDF
materials.xacro was xacro:included from both irb2600_macro.xacro and
spray_nozzle.xacro, which are both pulled into irb2600.urdf.xacro. xacro
does not deduplicate repeated includes of the same file, so the
'abb_orange' <material> definition ended up twice in the expanded URDF,
which urdfdom rejects ("material 'abb_orange' is not unique").

Fix: include materials.xacro exactly once, from the top-level assembly
file, before the macro files that reference it.

Reported when running `ros2 launch irb2600_description display.launch.py`
on Ubuntu 22.04 + ROS 2 Humble.

Co-Authored-By: Claude Sonnet 5 <noreply@anthropic.com>
Claude-Session: https://claude.ai/code/session_013pbvqy8ksWg6M6nbzUNzZ7

File: ros2_ws/src/irb2600_description/urdf/irb2600.urdf.xacro (robot description, xacro)
@@ -10,4 +10,12 @@
   -->
   <link name="world"/>
+  <!--
+    materials.xacro is included exactly once, here, before anything that
+    uses xacro:material_abb_orange. xacro does not deduplicate repeated
+    xacro:include of the same file, and urdfdom rejects a <material> name
+    that is defined (i.e. with a <color>/<texture> child) more than once --
+    so irb2600_macro.xacro and spray_nozzle.xacro must NOT also include it.
+  -->
+  <xacro:include filename="$(find irb2600_description)/urdf/materials.xacro"/>
   <xacro:include filename="$(find irb2600_description)/urdf/irb2600_macro.xacro"/>
   <xacro:include filename="$(find irb2600_description)/urdf/robot_base.xacro"/>

File: ros2_ws/src/irb2600_description/urdf/irb2600_macro.xacro (robot description, xacro)
@@ -1,5 +1,11 @@
 <?xml version="1.0" encoding="UTF-8"?>
 <robot xmlns:xacro="http://ros.org/wiki/xacro">
-  <xacro:include filename="$(find irb2600_description)/urdf/materials.xacro"/>
+  <!--
+    Note: does NOT xacro:include materials.xacro here -- it must be included
+    exactly once by whichever top-level file assembles the robot (see
+    irb2600.urdf.xacro), otherwise urdfdom rejects the duplicated
+    'abb_orange' material definition. This file only uses the
+    material_abb_orange macro, assuming it is already defined.
+  -->
   <!--
     ROS 2 port of RAMEL-ESPOL/IRB2600-ABB irb2600_description/urdf/irb2600_macro.xacro.

File: ros2_ws/src/irb2600_description/urdf/spray_nozzle.xacro (robot description, xacro)
@@ -17,5 +17,11 @@
                            encoded as a fixed offset here.
   -->
-  <xacro:include filename="$(find irb2600_description)/urdf/materials.xacro"/>
+  <!--
+    Note: does NOT xacro:include materials.xacro here -- it must be included
+    exactly once by whichever top-level file assembles the robot (see
+    irb2600.urdf.xacro), otherwise urdfdom rejects the duplicated
+    'abb_orange' material definition. This file only uses the
+    material_abb_orange macro, assuming it is already defined.
+  -->
   <link name="spray_nozzle_link">
     <inertial>
